File: Micro-mouse Project.kicad_sch (KiCad schematic)
At the start: 10 parts, among them U1 DRV8833PWPR

Commit message: Add files via upload
Parts:
- removed C1, C2, C?: C, symbol Device:C
- removed R1, R2, R?: R_Small_US, symbol Device:R_Small_US
- removed U1, U?: DRV8833PWPR, Package_SO:HTSSOP-16-1EP_4.4x5mm_P0.65mm_EP3.4x5mm_Mask2.46x2.31mm_ThermalVias, symbol Driver_Motor:DRV8833PWP
- added C1: 680uF, Capacitor_THT:CP_Axial_L18.0mm_D10.0mm_P25.00mm_Horizontal, symbol Device:C_Small
- added C12, C26: 100μF, Capacitor_SMD:C_1206_3216Metric_Pad1.33x1.80mm_HandSolder, symbol Device:C_Small
- added C14: 100nF, Capacitor_SMD:C_0402_1005Metric_Pad0.74x0.62mm_HandSolder, symbol Device:C_Small
- added C19: 10nF, Capacitor_SMD:C_0805_2012Metric_Pad1.18x1.45mm_HandSolder, symbol Device:C_Small
- added C21: 10μF, Capacitor_SMD:C_1206_3216Metric_Pad1.33x1.80mm_HandSolder, symbol Device:C_Small
- added C32, C33: 10μF, Capacitor_SMD:C_0805_2012Metric_Pad1.18x1.45mm_HandSolder, symbol Device:C_Small
- added D2: 1N5822, Library:DIO_SS34, symbol Diode:1N5822
- added IC1: CH224K, Library:SOP100P600X180-11N, symbol CH224K:CH224K
- added J3: USB_C_Receptacle_USB2.0_16P, Connector_USB:USB_C_Receptacle_GCT_USB4105-xx-A_16P_TopMnt_Horizontal, symbol Connector:USB_C_Receptacle_USB2.0_16P
- added L1: 33μH, Inductor_THT:L_Axial_L20.0mm_D8.0mm_P25.40mm_Horizontal, symbol Device:L_Small
- added Q2: 2N3904, Package_TO_SOT_SMD:SOT-23, symbol Transistor_BJT:2N3904
- added R10: 6.8k, Resistor_SMD:R_0603_1608Metric_Pad0.98x0.95mm_HandSolder, symbol Device:R_Small
- added R11: 4.7k, Resistor_SMD:R_0603_1608Metric_Pad0.98x0.95mm_HandSolder, symbol Device:R_Small
- added R12, R13, R21: 1k, Resistor_SMD:R_1206_3216Metric_Pad1.30x1.75mm_HandSolder, symbol Device:R_Small
- added R18: 5K, Resistor_SMD:R_0603_1608Metric, symbol Device:R_Small
- added R19: 10k, Resistor_SMD:R_0805_2012Metric_Pad1.20x1.40mm_HandSolder, symbol Device:R_Small
- added R20: 2.5K, Resistor_SMD:R_0603_1608Metric, symbol Device:R_Small
- added R4: 0.15, Resistor_SMD:R_1206_3216Metric_Pad1.30x1.75mm_HandSolder, symbol Device:R_Small
- added R6: 4.7K, Resistor_SMD:R_0603_1608Metric_Pad0.98x0.95mm_HandSolder, symbol Device:R_Small
- added TP1, TP2: TestPoint, symbol Connector:TestPoint
- added U2: LM2596S-5, Package_TO_SOT_SMD:TO-263-5_TabPin3, symbol Regulator_Switching:LM2596S-5
- added U7: TP4056-42-ESOP8, Library:SOIC127P600X175-9N, symbol Battery_Management:TP4056-42-ESOP8
- J1: renamed from J?; footprint (none) -> Connector_PinHeader_2.54mm:PinHeader_2x16_P2.54mm_Vertical
- U4: renamed from U?; footprint Package_SO:SOIC-8_3.9x4.9mm_P1.27mm -> Library:SOT65P280X145-8N; LCSC (none) -> C87469
Connections:
- net 3V3 Out: now also U4.1 (A1), U4.5 (VS), C14.2, R11.1, R6.1
- net Battery: now also U4.8 (IN+), C19.2, R4.1, U7.5 (BAT)
- net FAST_CHARGE_CTRL: now also Q2.2 (B)
- net GND: now also U4.2 (A0), U4.6 (GND), U4.7 (IN-), C1.2, C12.2, C14.1, C19.1, C21.1, C26.2, C32.2, C33.2, D2.2 (A), IC1.11 (GND), J3.A1 (GND), J3.A12 (GND), J3.B1 (GND), J3.B12 (GND), Q2.1 (E), R10.2, R18.2, R20.1, R4.2, U2.3 (GND), U2.5 (~{ON}/OFF), U7.1 (TEMP), U7.3 (GND), U7.9 (EPAD)
- net I2C1_SCL: now also U4.4 (SCL), R11.2
- net I2C1_SDA: now also U4.3 (SDA), R6.2
- net HV renamed High Voltage (9V)
- net High Voltage (9V): now also C1.1, R19.2, TP1.1, U2.1 (VIN)
- new net: C12.1, C21.2, C26.1, C32.1, C33.1, L1.2, R13.2, R21.2, TP2.1, U2.4 (FB), U7.4 (V_{CC}), U7.8 (CE)
- new net: D2.1 (K), L1.1, U2.2 (OUT)
- new net: R21.1, U7.7 (~{CHRG})
- new net: Q2.3 (C), R18.1, R20.2, U7.2 (PROG)
- new net: IC1.9 (CFG1), R10.1
- new net: IC1.7 (CC1), J3.A5 (CC1)
- new net: IC1.5 (DM), J3.A6 (D+), J3.B6 (D+)
- new net: IC1.4 (DP), J3.A7 (D-), J3.B7 (D-)
- new net: IC1.6 (CC2), J3.B5 (CC2)
- new net: IC1.8 (VBUS), R19.1
- new net: R13.1, U7.6 (~{STDBY})
- new net VDD: IC1.1 (VDD), R12.2
- new net Vbus: J3.A4 (VBUS), J3.A9 (VBUS), J3.B4 (VBUS), J3.B9 (VBUS), R12.1
- no-connect marks 0 -> 7
Other:
- note added: "BATTERY CHARGER CIRCUIT"
- note added: "BATTERY MONITOR CIRCUIT"
- note added: "Electrical pinout of the MM Power PCB"
- note added: "Our mouth of the circuit, connected too the high voltage pin of the pin header"
- note added: "PCB CONNECTOR"
- note added: "The charging IC that we connect the battery to With changing modes of charging with the NPN(2N3904)"
- note added: "This is an INA219 connected in the the 2*16 pin header, with pin A1 connected to the 3.3V out pin in and A0 connected to ground."
- note added: "This is the part of the circuit Receiving input from the output Of the CH224K and is stepped down to 5V"
- note added: "USB_C +9V INPUT"
- company: (none) -> Universiy of Cape Town
- title: (none) -> GRP 14 POWER SUB-SYSTEM
- moved on the sheet: J1, U4
